File: hardware/picozorro-one-th/picozorro-one-th.kicad_pcb (KiCad board)
At the start: 2 copper layers, 155.5 x 65.9 mm, 25 parts, among them J1 Zorro_II_Edge_100, J2 USB_A, J3 USB int, J4 SWD, J5 RUN/BOOT, M1J1 W5500 Lite J1, M1J2 W5500 Lite J2, M2 microSD breakout, M3J1 GY-PCM5102 6-pin, M3J2 GY-PCM5102 9-pin, P1 Core2350B P1, P2 Core2350B P2, P3 Core2350B P3, P4 Core2350B P4, Q1 2N3904, U2 LD1117V33

Commit message: One TH: SMD alternates for a JLC-assembled build, power block reworked
One board, two builds. The default build stays all through-hole; the
KiCad variant JLC fits an SMD alternate on the same nets for every
through-hole part: SS14, 1812 PTC, MMBT3904, 0603 resistors, an
AMS1117-3.3 under the TO-220, 22 uF MLCC banks under the electrolytics
and a Hirose microSD socket in place of the breakout. The silk frames
each pair with one label.

Power: U2 supplies 3V3_AUX in both builds, JP2 is the fallback without
it, C3 is 10 uF. Bus routing unchanged.

The 3D models carry KiCad's own sockets and jack; the DAC model is the
project's own, which drops the GPL zynthian STEP. Fab files add the JLC
BOM and placement list and order notes for both builds.
Parts:
- added C101: 22u, Capacitor_SMD:C_1206_3216Metric, F.Cu at (147.7, 102.8)
- added C102: 22u, Capacitor_SMD:C_1206_3216Metric, F.Cu at (150.1, 102.8)
- added C103: 22u, Capacitor_SMD:C_1206_3216Metric, F.Cu at (152.5, 102.8)
- added C201: 22u, Capacitor_SMD:C_1206_3216Metric, F.Cu at (162.4, 102.8)
- added C202: 22u, Capacitor_SMD:C_1206_3216Metric, F.Cu at (164.8, 102.8)
- added C203: 22u, Capacitor_SMD:C_1206_3216Metric, F.Cu at (167.2, 102.8)
- added C204: 22u, Capacitor_SMD:C_1206_3216Metric, F.Cu at (169.6, 102.8)
- added C205: 22u, Capacitor_SMD:C_1206_3216Metric, F.Cu at (172.0, 102.8)
- added C301: 10u, Capacitor_SMD:C_0805_2012Metric, F.Cu at (141.9, 87.4)
- added C401: 22u, Capacitor_SMD:C_1206_3216Metric, F.Cu at (137.1, 82.2)
- added C5: 100n, Capacitor_SMD:C_0603_1608Metric, F.Cu at (142.9, 64.4)
- added C6: 10u, Capacitor_SMD:C_0805_2012Metric, F.Cu at (159.9, 74.4)
- added D101: SS14, Diode_SMD:D_SMA, F.Cu at (158.0, 98.2)
- added F101: PTC 1.1A hold, Fuse:Fuse_1812_4532Metric, F.Cu at (167.1, 83.9)
- added J6: DM3AT-SF-PEJM5, Connector_Card:microSD_HC_Hirose_DM3AT-SF-PEJM5, F.Cu at (151.6, 63.5)
- added Q101: MMBT3904, Package_TO_SOT_SMD:SOT-23, F.Cu at (133.6, 92.8)
- added R101: 2.2k, Resistor_SMD:R_0603_1608Metric, F.Cu at (125.3, 93.9)
- added R2: 10k, Resistor_SMD:R_0603_1608Metric, F.Cu at (142.9, 70.5)
- added R3: 10k, Resistor_SMD:R_0603_1608Metric, F.Cu at (142.9, 67.5)
- added R4: 10k, Resistor_SMD:R_0603_1608Metric, F.Cu at (142.9, 61.4)
- added R5: 10k, Resistor_SMD:R_0603_1608Metric, F.Cu at (142.9, 58.4)
- added R6: 1R0, Resistor_SMD:R_0603_1608Metric, F.Cu at (137.1, 86.1)
- added U201: AMS1117-3.3, Package_TO_SOT_SMD:SOT-223-3_TabPin2, F.Cu at (122.8, 81.8)
- C3: value 100n -> 10u; footprint Capacitor_THT:C_Disc_D5.1mm_W3.2mm_P5.00mm -> Capacitor_THT:CP_Radial_D5.0mm_P2.00mm
- JP2: footprint Jumper:SolderJumper-2_P1.3mm_Bridged_RoundedPad1.0x1.5mm -> Jumper:SolderJumper-2_P1.3mm_Open_RoundedPad1.0x1.5mm
- moved D1 11.6 mm to (158.0, 93.1), turned to -90 degrees
- moved C1 4.66 mm to (148.8, 93.1)
- moved C3 1.55 mm to (141.0, 84.6)
- moved C2 1.45 mm to (165.4, 93.1)
- moved C4 0.60 mm to (133.8, 86.1)
Connections:
- net Net-(JP1-C) renamed INT_COLL
- net Net-(Q1-B) renamed INT_BASE
Routing:
- net 3V3_AUX: track 99.0 -> 145.4 mm, vias 1 -> 2
- net +5V: track 100.9 -> 128.1 mm, vias 2 -> 0
- net SD_DAT1: track 0.00 -> 25.6 mm
- net SPI1_MISO: track 77.9 -> 102.3 mm
- net VBUS_PORT: track 40.1 -> 57.7 mm
- net SPI1_MOSI: track 102.7 -> 116.8 mm
- net INT_COLL: track 16.5 -> 25.7 mm
- net SD_DAT2: track 0.00 -> 8.51 mm
- net GND: track 33.3 -> 39.3 mm, vias 258 -> 243
- net INT_BASE: track 9.03 -> 14.3 mm
- net SD_CS: track 81.0 -> 86.3 mm
- net INT_DRV: track 43.8 -> 48.0 mm
- net VIN: track 125.6 -> 122.6 mm, vias 4 -> 2
- net SPI1_SCK: track 95.6 -> 98.5 mm
- net CFGOUT: track 77.1 -> 75.2 mm
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Other:
- board text added: "C3 10u"
- board text added: "C4 10u"
- board text added: "Core2350B0"
- board text added: "JP2 3V3: bridge only without U2"
- board text added: "SMD"
- board text added: "U2 LD1117V33"
- board text removed: "C3 100n opt"
- board text removed: "C4 10u opt"
- board text removed: "Core2350B"
- board text removed: "JP2 3V3 (cut: U2)"
- board text removed: "U2 LD1117V33 opt: cut JP2"
