File: hardware/picozorro-one-th/picozorro-one-th.kicad_sch (KiCad schematic)
At the start: 25 parts, among them J1 Zorro_II_Edge_100, J2 USB_A, J3 USB int, J4 SWD, J5 RUN/BOOT, M1J1 W5500 Lite J1, M1J2 W5500 Lite J2, M2 microSD breakout, M3J1 GY-PCM5102 6-pin, M3J2 GY-PCM5102 9-pin, P1 Core2350B P1, P2 Core2350B P2, P3 Core2350B P3, P4 Core2350B P4, Q1 2N3904, U2 LD1117V33

Commit message: One TH: SMD alternates for a JLC-assembled build, power block reworked
One board, two builds. The default build stays all through-hole; the
KiCad variant JLC fits an SMD alternate on the same nets for every
through-hole part: SS14, 1812 PTC, MMBT3904, 0603 resistors, an
AMS1117-3.3 under the TO-220, 22 uF MLCC banks under the electrolytics
and a Hirose microSD socket in place of the breakout. The silk frames
each pair with one label.

Power: U2 supplies 3V3_AUX in both builds, JP2 is the fallback without
it, C3 is 10 uF. Bus routing unchanged.

The 3D models carry KiCad's own sockets and jack; the DAC model is the
project's own, which drops the GPL zynthian STEP. Fab files add the JLC
BOM and placement list and order notes for both builds.
Parts:
- added C101, C102, C103, C201, C202, C203, C204, C205, C401: 22u, Capacitor_SMD:C_1206_3216Metric, symbol Device:C_Small
- added C301, C6: 10u, Capacitor_SMD:C_0805_2012Metric, symbol Device:C_Small
- added C5: 100n, Capacitor_SMD:C_0603_1608Metric, symbol Device:C_Small
- added D101: SS14, Diode_SMD:D_SMA, symbol Device:D_Schottky_Small
- added F101: PTC 1.1A hold, Fuse:Fuse_1812_4532Metric, symbol Device:Polyfuse_Small
- added J6: DM3AT-SF-PEJM5, Connector_Card:microSD_HC_Hirose_DM3AT-SF-PEJM5, symbol Connector:Micro_SD_Card_Det_Hirose_DM3AT
- added Q101: MMBT3904, Package_TO_SOT_SMD:SOT-23, symbol Transistor_BJT:MMBT3904
- added R101: 2.2k, Resistor_SMD:R_0603_1608Metric, symbol Device:R_Small
- added R2, R3, R4, R5: 10k, Resistor_SMD:R_0603_1608Metric, symbol Device:R_Small
- added R6: 1R0, Resistor_SMD:R_0603_1608Metric, symbol Device:R_Small
- added U201: AMS1117-3.3, Package_TO_SOT_SMD:SOT-223-3_TabPin2, symbol Regulator_Linear:AMS1117-3.3
- C1, C2, D1, F1, M2, Q1, R1: Build (none) -> DIY
- C3: value 100n -> 10u; footprint Capacitor_THT:C_Disc_D5.1mm_W3.2mm_P5.00mm -> Capacitor_THT:CP_Radial_D5.0mm_P2.00mm; symbol Device:C_Small -> Device:C_Polarized_Small; Build (none) -> DIY; now fitted
- C4, U2: Build (none) -> DIY; now fitted
- JP2: footprint Jumper:SolderJumper-2_P1.3mm_Bridged_RoundedPad1.0x1.5mm -> Jumper:SolderJumper-2_P1.3mm_Open_RoundedPad1.0x1.5mm; symbol Jumper:SolderJumper_2_Bridged -> Jumper:SolderJumper_2_Open
Connections:
- net +5V: now also C101.1, C102.1, C103.1, C301.1, D101.2 (A), F101.1, U201.3 (VI)
- net 3V3_AUX: now also C5.1, C6.1, J6.4 (VDD), R2.1, R3.1, R4.1, R5.1, R6.1, U201.2 (VO)
- net GND: now also C101.2, C102.2, C103.2, C201.2, C202.2, C203.2, C204.2, C205.2, C301.2, C401.2, C5.2, C6.2, J6.6 (VSS), J6.SH (SHIELD), Q101.2 (E), U201.1 (GND)
- net INT_DRV: now also R101.1
- net SD_CS: now also J6.2 (DAT3/CD)
- net SPI1_MISO: now also J6.7 (DAT0), R4.2
- net SPI1_MOSI: now also J6.3 (CMD), R3.2
- net SPI1_SCK: now also J6.5 (CLK)
- net VBUS_PORT: now also C201.1, C202.1, C203.1, C204.1, C205.1, F101.2
- net VIN: now also D101.1 (K)
- net INT_COLL: now reaches JP1.2 (C), Q1.3 (C)
- net INT_COLL: now also Q101.3 (C)
- net INT_BASE: now reaches Q1.2 (B), R1.2
- net INT_BASE: now also Q101.1 (B), R101.2
- new net: C401.1, R6.2
- new net SD_DAT1: J6.8 (DAT1), R5.2
- new net SD_DAT2: J6.1 (DAT2), R2.2
- no-connect marks 57 -> 59
Other:
- note added: "11a. JLC build: SMD alternates of the power and interrupt parts"
- note added: "11b. JLC build: microSD socket J6 (replaces M2)"
- note added: "C101-C103: bulk on the bus +5V (C1). C201-C205: port bulk (C2). 22 uF 25 V X5R 1206, 13.6 uF each at 5 V."
- note added: "DIY build (default variant): U1, M1, D1, F1, C1, C2, Q1, R1, J2 or J3. Optional: M2 (microSD), M3 (DAC). U2, C3, C4 fitted (3V3_AUX regulator; JP2 open). Not fitted (DNP): J4 (developers), J5 (recovery). JLC build (variant JLC): the SMD parts of block 11 instead of D1, F1, C1-C4, Q1, R1, U2 and M2; modules, headers and J2 or J3 by hand. No pull-up on SD_CS (GPIO18). Bus signals only on GPIO0-38 (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"
- note added: "Hirose DM3AT-SF-PEJM5, push-push, under M2's outline, card detect open. CS = DAT3, MOSI = CMD, MISO = DAT0."
- note added: "JP2 OPEN as delivered. Bridge it only on a board without U2: +3V3 (U1 P2.16, module LDO) then feeds 3V3_AUX (M1, M2). U2 is fitted by default: JP2 stays open."
- note added: "M1 is fitted. RSTn stays open: the module has its own power-on reset (10k, 100 nF, 1N4148) and the firmware resets the W5500 in software. The module has 10k pull-ups on SCSn and INTn, so the W5500 is deselected while the RP2350 is in reset. INTn shares GPIO39 with the module's LED1. 3.3V from 3V3_AUX: U2 (default) or, without U2, the module LDO through JP2 (132 mA typical). Seated about 17.8 mm a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"
- note added: "Pull-ups, none on CS (as M2): R2 DAT2, R3 CMD (MOSI), R4 DAT0 (MISO), R5 DAT1: 10k to 3V3_AUX. C5 100 nF + C6 10 uF at the socket's VDD. DET_A / DET_B (9, 10) open. M2 (breakout) and J6 are never both fitted."
- note added: "Q101 SOT-23: 1 B, 2 E, 3 C (Q1 TO-92: 1 E, 2 B, 3 C)."
- note added: "Same nets as the through-hole part: D101 = D1 (SMD), C101-C103 = C1 (SMD), ... (number x 100 + n). The DIY build fits the through-hole parts (default variant), the JLC build these (variant JLC). Never both: the pads share the footprint area."
- note added: "U201: tab = VOUT, as U2. R6 in series with C401 gives the 22 uF MLCC the ESR of the tantalum the AMS1117 data sheet is written for."
- note added: "goes to J1 75 J1 77 J1 79 J1 81 J1 83 J1 86 J1 84 J1 82 J1 80 J1 78 J1 76 J1 71 J1 69 J1 67 J1 65 J1 63 J1 74 J1 72 M2.2 / J6.2 J1 68 J1 29 J1 27 J1 26 J1 24 J1 21 J1 23 J1 28 J1 18 J1 45 J1 47 J1 52 J1 54 J1 56 J1 58 J1 57 J1 59 J1 12 J1 11 J1 94 M1J1.6 M1J2.6, M2.5 / J6.7 M1J1.5 M1J1.4, M2.4 / J6.5 M1J1.3, M2.3 / J6.3 M3J1.3 R1 / R101 (Q1 base) M3J1.2 M3J1.4"
- note removed: "Fitted: U1, M1, D1, F1, C1, C2, Q1, R1, J2 or J3. Optional: M2 (microSD), M3 (DAC). Not fitted (DNP): U2, C3, C4 (fallback), J4 (developers), J5 (recovery). No pull-up on SD_CS (GPIO18). Bus signals only on GPIO0-38 (5 V tolerant); GPIO39-47 never see the bus. J1 70 (/LDS) is not connected on this board."
- note removed: "JP2 bridged as delivered: +3V3 (U1 P2.16, module LDO) feeds 3V3_AUX (M1, M2). Cut it when U2 is fitted."
- note removed: "M1 is fitted. RSTn stays open: the module has its own power-on reset (10k, 100 nF, 1N4148) and the firmware resets the W5500 in software. The module has 10k pull-ups on SCSn and INTn, so the W5500 is deselected while the RP2350 is in reset. INTn shares GPIO39 with the module's LED1. 3.3V from 3V3_AUX: the module LDO through JP2 (132 mA typical). Seated about 17.8 mm above the PCB on its header pl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"
- note removed: "goes to J1 75 J1 77 J1 79 J1 81 J1 83 J1 86 J1 84 J1 82 J1 80 J1 78 J1 76 J1 71 J1 69 J1 67 J1 65 J1 63 J1 74 J1 72 M2.2 J1 68 J1 29 J1 27 J1 26 J1 24 J1 21 J1 23 J1 28 J1 18 J1 45 J1 47 J1 52 J1 54 J1 56 J1 58 J1 57 J1 59 J1 12 J1 11 J1 94 M1J1.6 M1J2.6, M2.5 M1J1.5 M1J1.4, M2.4 M1J1.3, M2.3 M3J1.3 R1 (Q1 base) M3J1.2 M3J1.4"
